Commit message: cambio limites del joint_3
Para que no colisione con otro joint

File: robot_arm_urdf/urdf/robot_arm_urdf.urdf (robot description, URDF)
Before this commit: robot robot_arm_urdf, 9 links, 8 joints
Joints:
- joint joint_3: limit lower=0 upper=3.142 effort=200 velocity=3 -> lower=-1.572 upper=1.0 effort=200 velocity=3

Commit message: fix: mass de hand

File: robot_arm_urdf/urdf/robot_arm_urdf.urdf (robot description, URDF)
Before this commit: robot robot_arm_urdf, 9 links, 8 joints
Links:
- link link_6: mass 0.11653 -> 0.51653
- link link_7: mass 0.11653 -> 0.51653
